Commit message: Publish transformations btw frames
Publish static transformations between inertial_NWU-inertial_NED and body_FLU-body_FRD.
Publish non-static transformation between inertial_NWU-body_FRU to connect model with global axis.
All transforms are published in model plugin.

File: last_letter_2/models/aircraft/plane.urdf (robot description, URDF)
Before this commit: robot plane, 8 links, 7 joints
Links:
- removed link body
- added link body_FLU, mass 2; collision cylinder length=2.5 radius=0.5; visual cylinder length=2.5 radius=0.5
Joints:
- removed joint  body_to_wheel_base
- removed joint bodyToWing
- removed joint body_to_arm
- removed joint body_to_rear_wheel
- added joint  body_FLU_to_wheel_base: type revolute, parent body_FLU, child wheel_base, origin xyz=1 0 -0.5 rpy=0 0 0, limit lower=-0.00872665 upper=0.00872665 effort=10.0 velocity=0.5
- added joint body_FLUToWing: type revolute, parent body_FLU, child airfoil, origin xyz=0.3 0 0.4 rpy=3.14 0 0, limit lower=-0.00872665 upper=0.00872665 effort=1000.0 velocity=0.5
- added joint body_FLU_to_arm: type continuous, parent body_FLU, child arm, origin xyz=1.25 0 0 rpy=0 1.57  0, axis 0 0 1
- added joint body_FLU_to_rear_wheel: type continuous, parent body_FLU, child rear_wheel, origin xyz=-1 0 -0.5, axis 0 1 0

File: last_letter_2/models/aircraft/plane.urdf.xacro (robot description, xacro)
@@ -1,4 +1,4 @@
 <robot name="plane" xmlns:xacro="http://www.ros.org/wiki/xacro">
-    <link name="body">
+    <link name="body_FLU">
         <visual>
             <origin rpy="0 -1.57 0 " />
@@ -38,7 +38,7 @@
         </inertial>
     </link>
-    <joint name="bodyToWing" type="revolute">
+    <joint name="body_FLUToWing" type="revolute">
         <origin xyz="0 0 0" rpy ="0 0 0"/>
-        <parent link="body" />
+        <parent link="body_FLU" />
         <child link="airfoil" />
         <limit effort="1000.0" lower="-0.000872665" upper="0.000872665" velocity="0.5"/>
@@ -65,8 +65,8 @@
         </inertial>
     </link>
-    <joint name="body_to_arm" type="continuous">
+    <joint name="body_FLU_to_arm" type="continuous">
         <origin xyz="1.25 0 0" rpy="0 1.57  0" />
         <axis xyz="0 0 1" />
-        <parent link="body" />
+        <parent link="body_FLU" />
         <child link="arm" />
     </joint>
@@ -111,7 +111,7 @@
         </inertial>
     </link>
-    <joint name=" body_to_wheel_base" type="fixed">
+    <joint name=" body_FLU_to_wheel_base" type="fixed">
         <origin xyz="1 0 -0.5" rpy="0 0 0" />
-        <parent link="body" />
+        <parent link="body_FLU" />
         <child link="wheel_base" />
     </joint>
@@ -186,8 +186,8 @@
         </inertial>
     </link>
-    <joint name="body_to_rear_wheel" type="continuous">
+    <joint name="body_FLU_to_rear_wheel" type="continuous">
         <origin xyz="-1 0 -0.5" />
         <axis xyz="0 1 0"/>
-        <parent link="body" />
+        <parent link="body_FLU" />
         <child link="rear_wheel" />
     </joint>
@@ -195,5 +195,5 @@
     <plugin name="model_plugin" filename="libmodel_plugin.so"/>
     <plugin name="joint_state_publisher" filename="libgazebo_ros_joint_state_publisher.so">
-        <jointName>bodyToWing, body_to_arm, wheel_base_to_left_wheel, wheel_base_to_right_wheel, body_to_rear_wheel </jointName>
+        <jointName>body_FLUToWing, body_FLU_to_arm, wheel_base_to_left_wheel, wheel_base_to_right_wheel, body_FLU_to_rear_wheel </jointName>
         <robotNamespace>last_letter_2</robotNamespace>
         <updateRate>0</updateRate>
