Commit message: Rotate wind vector
Transform wind vector exported from body frame, to motor frame.

File: last_letter_2/config/param/aircrafts/csl_2k19/urdf/model.urdf.xacro (robot description, xacro)
@@ -16,5 +16,5 @@
             </geometry>
         </visual>
-        <collision>kids
+        <collision>
             <origin rpy="0 -${pi/2} 0 " />
             <geometry>
